File: Electronics/Infrared/ProximitySensor.sch (EAGLE design)
At the start: 9 parts, among them IC1 LM358D

Commit message: modification de la carte (trimmer CMS en trimmer THT)
Parts:
- R1: device rcl:R-TRIMM4G/J -> rcl:R-TRIMMT93YA
Changed lines of the file:
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@@
 <parts>
 <part name="IC1" library="linear" deviceset="LM358" device="D" value="LM358D"/>
-<part name="R1" library="rcl" deviceset="R-TRIMM" device="4G/J"/>
+<part name="R1" library="rcl" deviceset="R-TRIMM" device="T93YA"/>
 <part name="LED_IR" library="led" deviceset="SFH482" device=""/>
 <part name="P+1" library="supply1" deviceset="VCC" device=""/>
